File: serial-port/serial.sch (KiCad schematic (older format))
At the start: 20 parts, among them J1 12V Pwr, J2 Serial 5V, J3 XL-320, J4 AX-12A, U1 AP1117-50, U2 LM317, U3 74LS126

Commit message: serial port fixes
Parts:
- added Q1, Q2: BSS138, TO_SOT_Packages_SMD:SOT-23, symbol BSS138
- added R10, R6, R8, R9: 10k, Resistors_SMD:R_1206_HandSoldering, symbol R
- J2: value Serial 5V -> Serial; footprint Pin_Headers:Pin_Header_Straight_1x04_Pitch2.54mm -> Pin_Headers:Pin_Header_Straight_1x05_Pitch2.54mm; symbol Conn_01x04 -> Conn_01x05
- renumbered D3 to D1, D1 to D2, D2 to D3, R6 to R1, R1 to R2, R2 to R3, R3 to R4, R4 to R5, R5 to R7
Connections:
- net VCC is gone; now on net +5V: U3.14 (VCC), U3.14 (VCC), U3.14 (VCC), U3.14 (VCC)
- net +5V: now also R10.1, R8.1
- net DATA: now also U3.5 (D); no longer U3.2
- net DTR: now also J2.5 (Pin_5), U3.4 (E); no longer J2.2 (Pin_2), U3.1 (E)
- net RXI: now also U3.6 (O), Q1.3 (D), R8.2; no longer J2.4 (Pin_4), U3.3
- net TXO: now also Q2.3 (D), R10.2; no longer J2.3 (Pin_3)
- new net +3V3: J2.2 (Pin_2), R6.1, R9.1
- new net RXI3v3: J2.4 (Pin_4), Q1.1 (G), Q1.2 (S), R6.2
- new net TXO3v3: J2.3 (Pin_3), Q2.1 (G), Q2.2 (S), R9.2

Commit message: update
Parts:
- removed Q1, Q2: BSS138, TO_SOT_Packages_SMD:SOT-23, symbol BSS138
- added Q1, Q2: BS170, TO_SOT_Packages_THT:TO-92_Inline_Wide, symbol BS170
Connections:
- net RXI: now also Q1.1 (D)
- net RXI3v3: now also Q1.2 (G), Q1.3 (S)
- net TXO: now also Q2.1 (D)
- net TXO3v3: now also Q2.2 (G), Q2.3 (S)
Changed lines of the file:
@@
 	1    0    0    -1
-$EndComp
-$Comp
-L BSS138 Q1
-U 1 1 5A9B2E59
-P 8100 4400
-F 0 "Q1" H 8300 4475 50  0000 L CNN
-F 1 "BSS138" H 8300 4400 50  0000 L CNN
-F 2 "TO_SOT_Packages_SMD:SOT-23" H 8300 4325 50  0001 L CIN
-F 3 "" H 8100 4400 50  0001 L CNN
-	1    8100 4400
-	0    1    1    0
 $EndComp
 Text GLabel 8500 4500 2    60   Output ~ 0
@@
 	1    0    0    -1
 $EndComp
-$Comp
-L BSS138 Q2
-U 1 1 5A9B3CC4
-P 9750 4350
-F 0 "Q2" H 9950 4425 50  0000 L CNN
-F 1 "BSS138" H 9950 4350 50  0000 L CNN
-F 2 "TO_SOT_Packages_SMD:SOT-23" H 9950 4275 50  0001 L CIN
-F 3 "" H 9750 4350 50  0001 L CNN
-	1    9750 4350
-	0    1    1    0
-$EndComp
 Wire Wire Line
 	9350 4450 9550 4450
@@
 Text GLabel 5350 1150 2    60   Input ~ 0
 TXO3v3
+$Comp
+L BS170 Q1
+U 1 1 5A9CB1AE
+P 8100 4400
+F 0 "Q1" H 8300 4475 50  0000 L CNN
+F 1 "BS170" H 8300 4400 50  0000 L CNN
+F 2 "TO_SOT_Packages_THT:TO-92_Inline_Wide" H 8300 4325 50  0001 L CIN
+F 3 "" H 8100 4400 50  0001 L CNN
+	1    8100 4400
+	0    1    1    0
+$EndComp
+$Comp
+L BS170 Q2
+U 1 1 5A9CB504
+P 9750 4350
+F 0 "Q2" H 9950 4425 50  0000 L CNN
+F 1 "BS170" H 9950 4350 50  0000 L CNN
+F 2 "TO_SOT_Packages_THT:TO-92_Inline_Wide" H 9950 4275 50  0001 L CIN
+F 3 "" H 9750 4350 50  0001 L CNN
+	1    9750 4350
+	0    1    1    0
+$EndComp
 $EndSCHEMATC
