File: serial-port-v2/serial.kicad_pcb (KiCad board)
At the start: 2 copper layers, 49.5 x 45.7 mm, 30 parts, among them J1 12V Pwr, J2 Serial, J3 XL-320, J4 AX-12A, J5 XL-320, J6 AX-12A, Q1 BSS138, U1 AP1117-50, U2 LM317, U4 74LVC1G126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

Commit message: board fixes
Parts:
- moved J3 1.91 mm to (95.2, 48.3)
- moved J4 1.27 mm to (95.2, 33.0)
Connections:
- Q1 pad 1: Net-(Q1-Pad1) -> +3V3
- Q1 pad 2: Net-(Q1-Pad1) -> Net-(Q1-Pad2)
- R5 pad 2: Net-(Q1-Pad1) -> Net-(Q1-Pad2)
- U4 pad 2: Net-(Q1-Pad1) -> Net-(Q1-Pad2)
- U5 pad 4: Net-(Q1-Pad1) -> Net-(Q1-Pad2)
Routing:
- net Net-(Q1-Pad1): track 30.3 -> 0.00 mm
- net Net-(Q1-Pad2): track 0.00 -> 29.2 mm
- net DATA: track 44.1 -> 61.5 mm
- net +3V3: track 53.4 -> 67.3 mm, vias 4 -> 6
- net +12V: track 75.2 -> 68.6 mm, vias 1 -> 0
- net +8V: track 51.6 -> 52.3 mm, vias 1 -> 0
